Commit message: full urdf

File: dragon.urdf (robot description, URDF)
Before this commit: robot dragon, 18 links, 17 joints
Links:
- added link imu_link, mass 0.001; collision box size=.001 .001 .001; visual box size=0.001 0.001 0.001
- link body: mass 1.2 -> 9.9629698
- link left_back_leg: mass 0.12 -> 0.58240446
- link left_back_shine: mass 0.12 -> 0.29186134
- link left_back_upper: mass 0.001 -> 0.67833686
- link left_front_leg: mass 0.12 -> 0.58240446
- link left_front_shine: mass 0.12 -> 0.29186134
- link left_front_upper: mass 0.001 -> 0.67833686
- link right_back_leg: mass 0.12 -> 0.58240446
- link right_back_shine: mass 0.12 -> 0.29186134
- link right_back_upper: mass 0.001 -> 0.67833686
- link right_front_leg: mass 0.12 -> 0.58240446
- link right_front_shine: mass 0.12 -> 0.29186134
- link right_front_upper: mass 0.001 -> 0.67833686
Joints:
- added joint imu_joint: type revolute, parent body, child imu_link, origin xyz=0 0 0, limit lower=0 upper=0 effort=0 velocity=0
- joint left_back_hip: limit lower=-0.78539815 upper=0.698131689 effort=100 velocity=100 -> lower=-0.78539815 upper=0.698131689 effort=1000 velocity=100
- joint left_back_knee: limit lower=0.174532922 upper=1.919862144 effort=100 velocity=100 -> lower=0.174532922 upper=1.919862144 effort=1000 velocity=100
- joint left_front_hip: limit lower=-0.698131689 upper=0.78539815 effort=100 velocity=100 -> lower=-0.698131689 upper=0.78539815 effort=1000 velocity=100
- joint left_front_knee: limit lower=-1.919862144 upper=-0.174532922 effort=100 velocity=100 -> lower=-1.919862144 upper=-0.174532922 effort=1000 velocity=100
- joint right_back_hip: limit lower=-0.78539815 upper=0.698131689 effort=100 velocity=100 -> lower=-0.78539815 upper=0.698131689 effort=1000 velocity=100
- joint right_back_knee: limit lower=0.174532922 upper=1.919862144 effort=100 velocity=100 -> lower=0.174532922 upper=1.919862144 effort=1000 velocity=100
- joint right_front_hip: limit lower=-0.698131689 upper=0.78539815 effort=100 velocity=100 -> lower=-0.698131689 upper=0.78539815 effort=1000 velocity=100
- joint right_front_knee: limit lower=-1.919862144 upper=-0.174532922 effort=100 velocity=100 -> lower=-1.919862144 upper=-0.174532922 effort=1000 velocity=100
